File: lipoboard.kicad_sch (KiCad schematic)
At the start: 51 parts, among them J1 USB_C_Receptacle_PowerOnly_24P, SW1 SW_DIP_x01, U1 TPS2116DRL, U3 DW01A, U5 TPS63001

Commit message: Init!
Changed lines of the file:
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@@
 	(text "Priority Power MUX"
 		(exclude_from_sim no)
-		(at 250.19 14.478 0)
+		(at 240.538 14.986 0)
 		(effects
 			(font
@@
 	(text "Battery Charger"
 		(exclude_from_sim no)
-		(at 122.174 15.494 0)
+		(at 124.714 14.478 0)
 		(effects
 			(font

Commit message: Add readme
Parts:
- 3V1, 3V2, 3V3, 5V1, 5V2, 5V3, B+1, B-1, BT1, IN+1, IN-1, OUT+1, OUT-1: now left out of the parts list
- C1, C10, C2, C3, C4, C5, C7, C8, C9: LCSC (none) -> C1713
- C11: LCSC (none) -> C45783
- C12, C6: LCSC (none) -> C38141
- D1, D3: LCSC (none) -> C22371297
- D2: LCSC (none) -> C2286
- J1: LCSC (none) -> C18357553
- L1, L2: LCSC (none) -> C177244
- R1: LCSC (none) -> C247017
- R10: LCSC (none) -> C1359
- R11: value 100 -> 100Ω; LCSC (none) -> C17408
- R12: LCSC (none) -> C17616
- R13: LCSC (none) -> C17819
- R2, R3, R8: LCSC (none) -> C2907195
- R4, R6: LCSC (none) -> C2930296
- R5: LCSC (none) -> C2933524
- R7: LCSC (none) -> C25612
- R9: LCSC (none) -> C2907267
- SW1: LCSC (none) -> C126888
- U1: LCSC (none) -> C3235557
- U2: value ~ -> TP4056; LCSC (none) -> C725790
- U3: LCSC (none) -> C2927799
- U4: value ~ -> TP5188; LCSC (none) -> C29075512
- U5: footprint Package_SON:Texas_DRC0010J_ThermalVias -> Package_SON:Texas_DRC0010J; LCSC (none) -> C28060
- U6: value ~ -> 8025A; now left out of the parts list
Other:
- moved on the sheet: L1
