File: src/lipoboard.kicad_sch (KiCad schematic)
At the start: 51 parts, among them J1 USB_C_Receptacle_PowerOnly_24P, SW1 SW_DIP_x01, U1 TPS2116DRL, U2 TP4056, U3 DW01A, U4 TP5188, U5 TPS63001, U6 8025A

Commit message: Change dir structure
Parts:
- U3, U6: footprint Package_TO_SOT_SMD:SOT-23-6 -> Package_TO_SOT_SMD:SOT-23-6_Handsoldering
- U5: footprint Package_SON:Texas_DRC0010J -> Package_SON:Texas_DRC0010J_ThermalVias
Changed lines of the file:
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@@
 			)
 		)
-		(property "Footprint" "Package_TO_SOT_SMD:SOT-23-6"
+		(property "Footprint" "Package_TO_SOT_SMD:SOT-23-6_Handsoldering"
 			(at 60.96 86.36 0)
 			(effects
@@
 			)
 		)
-		(property "Footprint" "Package_TO_SOT_SMD:SOT-23-6"
+		(property "Footprint" "Package_TO_SOT_SMD:SOT-23-6_Handsoldering"
 			(at 60.96 105.41 0)
 			(effects
@@
 			)
 		)
-		(property "Footprint" "Package_SON:Texas_DRC0010J"
+		(property "Footprint" "Package_SON:Texas_DRC0010J_ThermalVias"
 			(at 255.27 111.76 0)
 			(effects
